File: ramiie.sch (KiCad schematic (older format))
At the start: 28 parts, among them J1 AppleIIeAux, U1 EPM7128SL84

Commit message: did a lot
Parts:
- removed C10, C14: 100n, Capacitor_SMD:C_0805_2012Metric, symbol Device:C_Small
- removed C16: 33u, stdpads:CP_EIA-3528, symbol Device:CP_Small
- removed FD5: Fiducial, stdpads:Fiducial, symbol Mechanical:MountingHole
- removed H5: (no value), stdpads:PasteHole_1.1mm_PTH, symbol Mechanical:MountingHole_Pad
- removed J?: Conn_01x08, symbol Connector_Generic:Conn_01x08
- removed J?: Conn_01x24, symbol Connector_Generic:Conn_01x24
- added R1: 100, symbol Device:R_Small
- C1, C2, C3, C4, C5, C6, C7, C8, C9: footprint Capacitor_SMD:C_0805_2012Metric -> stdpads:C_0805
- J1: footprint (none) -> stdpads:AppleIIeAux_Edge
- JP101: renamed from JP?; footprint (none) -> Connector_PinHeader_2.54mm:PinHeader_1x02_P2.54mm_Vertical_SMD_Pin1Left
- U1: footprint (none) -> stdpads:PLCC-84; symbol StandardParts:EPM7128SL84 -> stdparts:EPM7128SL84
- U101: renamed from U?; footprint (none) -> stdpads:SOJ-28-300mil
- renumbered FD1 to FID1, FD2 to FID2, FD3 to FID3, FD4 to FID4
Connections:
- net labels added: RA11
- net labels removed: MA0, MA1, MA2, MA3, MA4, MA5, MA6, MA7
- wire segments 45 -> 36
- no-connect marks 1 -> 0
Other:
- moved on the sheet: JP101

Commit message: I think it's done
Parts:
- removed C9: 100n, stdpads:C_0805, symbol Device:C_Small
- removed JP101: Jumper_NO_Small, Connector_PinHeader_2.54mm:PinHeader_1x02_P2.54mm_Vertical_SMD_Pin1Left, symbol Device:Jumper_NO_Small
- removed R1: 100, symbol Device:R_Small
- renumbered U101 to U2
Connections:
- wire segments 36 -> 260
- no-connect marks 0 -> 4
Other:
- note added: "00000"
- note added: "00001"
- note added: "00011"
- note added: "01000"
- note added: "01011"
- note added: "01100"
- note added: "01111"
- note added: "10000"
- note added: "10011"
- note added: "10100"
- note added: "10111"
- note added: "11000"
- note added: "11001"
- note added: "11011"
- note added: "6502 CPU Access"
- note added: "C14M"
- note added: "C7M"
- note added: "GateCRAS"
- note added: "GateCRAS <= state == 10100 | 01111 | 00011 | 01011 @ C14M\nnRefRAS <= ~state == 01111 | 01011 | 00001~ @ C14M\nnRefCAS <= ~state == 01111 | 00011~ @ ~C14M~\nGateWE <= state == 10100 | 00011 @ C14M\nHoldRow <= state == 01011 | 10011 @ ~C14M~\n\nRowAddr[7:0] <= MA[7:0] @ ~nPRAS~\nBA[5:0] <= D[5:0] @ C14M in state == 10100 & RowAddr == 73 & C07X"
- note added: "GateWE"
- note added: "HoldRow"
- note added: "PHI0"
- note added: "Q3"
- note added: "VDR[7:0] <= RD[7:0] @ PHI0\nVD[7:0] <= PHI1 ? 8’bZ : VDR[7:0]\nD[7:0] <= (EN80 & R~W~80) ? RD[7:0] : 8’bZ\nRD[7:0] <= (EN80 & ~R~W80) ? D[7:0] : 8’bZ"
- note added: "Video Access"
- note added: "nCAS"
- note added: "nPCAS"
- note added: "nPRAS"
- note added: "nRAS"
- note added: "nRAS <= GateCRAS ? nRefRAS : nPRAS\nnCAS <= GateCRAS ? nRefCAS : Q3\nnRWE <= GateWE | RW80\nRA[7:0] <= HoldRow ? RowAddr[7:0] : MA[7:0]\nRA[10:8] <= PHI1 ? 0 : HoldRow ? BA[5:3] : BA[2:0]\nRA[11] <= PHI1 ? 0 : BA[5]"
- note added: "nRefCAS"
- note added: "nRefRAS"
- moved on the sheet: FID1, FID2, FID3, FID4, H1, H2, H3, H4, J1, U2
